File: Electrical/pcb/reflow_oven/Interfaces.kicad_sch (KiCad schematic)
At the start: 14 parts, among them P1 USB_C_Receptacle_USB2.0, U4 CP2102N-Axx-xQFN28

Commit message: interface
partial interface schematic
Parts:
- added C15: 100nF, Capacitor_SMD:C_0603_1608Metric, symbol Device:C
- added D7: SM712_SOT23, Package_TO_SOT_SMD:SOT-23, symbol Diode:SM712_SOT23
- added F3, F4: 300mA, Fuse:Fuse_1206_3216Metric_Pad1.42x1.75mm_HandSolder, symbol Device:Polyfuse
- added J3: DB9_Female, Connector_Dsub:DSUB-9_Female_Horizontal_P2.77x2.84mm_EdgePinOffset7.70mm_Housed_MountingHolesOffset9.12mm, symbol Connector:DB9_Female
- added R17, R18: 10K, Resistor_SMD:R_0603_1608Metric, symbol Device:R
- added R19, R20, R21, R22: 22, Resistor_SMD:R_0603_1608Metric, symbol Device:R
- added R23: 120, Resistor_SMD:R_0805_2012Metric_Pad1.20x1.40mm_HandSolder, symbol Device:R
- added U5: MAX485E, footprint_lib:SOIC127P600X175-8N, symbol Interface_UART:MAX485E
- renumbered R3 to R10, R4 to R11, R5 to R12, R6 to R13, R7 to R14, R8 to R15, R9 to R16
Connections:
- net +3V3: now also C15.1, R17.2, U5.8 (VCC)
- net GND: now also C15.2, D7.3 (common), J3.5, R18.1, U5.5 (GND)
- net RX: no longer names the net of R16.1, U4.25 (RXD)
- net RX_0 renamed RX_MCU_usb
- net TX: no longer names the net of R15.1, U4.26 (TXD)
- net TX_0 renamed TX_MCU_usb
- new net: F4.1, R23.1, U5.6 (A)
- new net: F3.1, R23.2, U5.7 (B)
- new net: R19.2, U5.1 (RO)
- new net: R20.2, U5.2 (~{RE})
- new net: R21.2, U5.3 (DE)
- new net: R22.2, U5.4 (DI)
- new net A: D7.1 (A1), F4.2, J3.7
- new net B: D7.2 (A2), F3.2, J3.3
- new net DE_485: R18.2, R21.1
- new net RX_MCU_485: R19.1
- new net TX_MCU_485: R22.1
- new net ~{RE}_485: R17.1, R20.1
- no-connect marks 20 -> 26
Other:
- note added: "DNP"
- note added: "RS-485"
- moved on the sheet: R15, R16

Commit message: analog Sensing
-voltage and current sensor
-zero crossing
-temperature
Parts:
- removed J3: DB9_Female, Connector_Dsub:DSUB-9_Female_Horizontal_P2.77x2.84mm_EdgePinOffset7.70mm_Housed_MountingHolesOffset9.12mm, symbol Connector:DB9_Female
- added J3: DB9_Female_MountingHoles, Connector_Dsub:DSUB-9_Female_Horizontal_P2.77x2.84mm_EdgePinOffset7.70mm_Housed_MountingHolesOffset9.12mm, symbol Connector:DB9_Female_MountingHoles
- renumbered C13 to C14, C14 to C15, C15 to C16, R10 to R13, R11 to R14, R12 to R15, R13 to R16, R14 to R17, R15 to R18, R16 to R19, R17 to R20, R18 to R21, R19 to R22, R20 to R23, R21 to R24, R22 to R25, R23 to R26
Connections:
- net A: now also J3.7
- net B: now also J3.3
- net GND: now also J3.0 (PAD), J3.5
Other:
- note added: "TODO - buttons, screen, buzzer"
- note removed: "TODO - usb to serial - rs485 compatible serial - buttons, screen, buzzer"

Commit message: schematic
-interface
-micro
todo
output
routing
Parts:
- added J3: USER BOARD DISPLAY, footprint_lib:SHDR10W66P254_2X5_2019X914X986P, symbol Connector_Generic:Conn_02x05_Odd_Even
- added J4: USER BOARD BUTTON, footprint_lib:SHDR10W66P254_2X5_2019X914X986P, symbol Connector_Generic:Conn_02x05_Odd_Even
- renumbered J3 to J5, R13 to R17, R14 to R18, R15 to R19, R16 to R20, R17 to R21, R18 to R22, R19 to R23, R20 to R24, R21 to R25, R22 to R26, R23 to R27, R24 to R28, R25 to R29, R26 to R30
Connections:
- net +3V3: now also J3.1 (Pin_1), J3.2 (Pin_2), J4.1 (Pin_1), J4.2 (Pin_2)
- net GND: now also J3.10 (Pin_10), J3.9 (Pin_9), J4.10 (Pin_10), J4.9 (Pin_9)
- new net BUZZER: J4.8 (Pin_8)
- new net DWN_BTN: J4.5 (Pin_5)
- new net I2C1_SCL: J3.7 (Pin_7)
- new net I2C1_SDA: J3.8 (Pin_8)
- new net LCD_CS: J3.6 (Pin_6)
- new net LCD_RST: J3.5 (Pin_5)
- new net LT_BTN: J4.4 (Pin_4)
- new net OK_BTN: J4.7 (Pin_7)
- new net RT_BTN: J4.6 (Pin_6)
- new net SPI2_CLK: J3.3 (Pin_3)
- new net SPI2_MOSI_RW: J3.4 (Pin_4)
- new net UP_BTN: J4.3 (Pin_3)
Other:
- note added: "User Board connector"
