File: Electrical/pcb/reflow_oven/Interfaces.kicad_sch (KiCad schematic)
At the start: 35 parts, among them J3 USER BOARD DISPLAY, J4 USER BOARD BUTTON, J5 DB9_Female_MountingHoles, P1 USB_C_Receptacle_USB2.0, U4 CP2102N-Axx-xQFN28, U5 MAX485E

Commit message: addon
documentation pics
adjust oshw logo
Parts:
- TP10, TP11, TP6, TP7, TP8, TP9: now left out of the parts list
Changed lines of the file:
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@@
   )
   (symbol (lib_id "Connector:TestPoint") (at 228.6 54.61 180) (unit 1)
-    (in_bom yes) (on_board yes)
+    (in_bom no) (on_board yes)
     (property "Reference" "TP9" (id 0) (at 231.14 59.69 0)
       (effects (font (size 1.27 1.27)) (justify left))
@@
   )
   (symbol (lib_id "Connector:TestPoint") (at 252.73 44.45 0) (unit 1)
-    (in_bom yes) (on_board yes)
+    (in_bom no) (on_board yes)
     (property "Reference" "TP10" (id 0) (at 251.46 39.37 0)
       (effects (font (size 1.27 1.27)) (justify left))
@@
   )
   (symbol (lib_id "Connector:TestPoint") (at 166.37 33.02 0) (unit 1)
-    (in_bom yes) (on_board yes)
+    (in_bom no) (on_board yes)
     (property "Reference" "TP6" (id 0) (at 165.1 27.94 0)
       (effects (font (size 1.27 1.27)) (justify left))
@@
   )
   (symbol (lib_id "Connector:TestPoint") (at 252.73 54.61 180) (unit 1)
-    (in_bom yes) (on_board yes)
+    (in_bom no) (on_board yes)
     (property "Reference" "TP11" (id 0) (at 254 59.69 0)
       (effects (font (size 1.27 1.27)) (justify left))
@@
   )
   (symbol (lib_id "Connector:TestPoint") (at 166.37 38.1 180) (unit 1)
-    (in_bom yes) (on_board yes)
+    (in_bom no) (on_board yes)
     (property "Reference" "TP7" (id 0) (at 168.91 43.18 0)
       (effects (font (size 1.27 1.27)) (justify left))
@@
   )
   (symbol (lib_id "Connector:TestPoint") (at 228.6 44.45 0) (unit 1)
-    (in_bom yes) (on_board yes)
+    (in_bom no) (on_board yes)
     (property "Reference" "TP8" (id 0) (at 227.33 39.37 0)
       (effects (font (size 1.27 1.27)) (justify left))
