File: Electrical/pcb/reflow_oven/Sensors.kicad_sch (KiCad schematic)
At the start: 87 parts, among them J10 THC IN, J11 THC IN, J12 NTC_A IN, J13 NTC_B IN, J6 Line IN, J7 Heater_A, J8 Line IN, J9 Heater_B, T1 ZMPT101B, T2 ZMPT101B, U10 TLP2361, U11 COS6001, U12 COS6001, U13 COS6001, U14 COS6001, U6 MAX6675ISA+T, U7 MAX6675ISA+T, U8 ACS758LCB-050B-PFF, U9 ACS758LCB-050B-PFF

Commit message: pcb layout
Parts:
- added TP?: Csense_A, symbol Connector:TestPoint
- added TP?: Csense_B, symbol Connector:TestPoint
- J7: value Heater_A -> Line IN
Connections:
- net CurrentSens_A: now also TP?.1
- net CurrentSens_B: now also TP?.1
- net at F6.1, U8.4 (IP+): now also J6.1 (Pin_2); no longer J6.2 (Pin_2)
- net at U8.5 (IP-): now also J7.2 (Pin_1); no longer J7.1 (Pin_1)
- new net: J6.2 (Pin_1), J7.1 (Pin_2), T1.2 (AB)
Changed lines of the file:
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@@
+    (stroke (width 0) (type default) (color 0 0 0 0))
+  )
+  (wire (pts (xy 114.3 92.71) (xy 114.3 95.25))
     (stroke (width 0) (type default) (color 0 0 0 0))
   )
@@
   )
   (wire (pts (xy 59.69 232.41) (xy 60.96 232.41))
+    (stroke (width 0) (type default) (color 0 0 0 0))
+  )
+  (wire (pts (xy 114.3 33.02) (xy 114.3 35.56))
     (stroke (width 0) (type default) (color 0 0 0 0))
   )
@@
     )
     (property "Datasheet" "" (id 3) (at 176.53 68.58 0)
+      (effects (font (size 1.27 1.27)) hide)
+    )
+    (pin "1")
+  )
+  (symbol (lib_id "Connector:TestPoint") (at 114.3 33.02 0) (unit 1)
+    (in_bom yes) (on_board yes)
+    (property "Reference" "TP?" (id 0) (at 113.03 27.94 0)
+      (effects (font (size 1.27 1.27)) (justify left))
+    )
+    (property "Value" "Csense_A" (id 1) (at 115.57 30.48 0)
+      (effects (font (size 1.27 1.27)) (justify left))
+    )
+    (property "Footprint" "" (id 2) (at 119.38 33.02 0)
+      (effects (font (size 1.27 1.27)) hide)
+    )
+    (property "Datasheet" "~" (id 3) (at 119.38 33.02 0)
       (effects (font (size 1.27 1.27)) hide)
     )
@@
     (pin "5")
   )
-  (symbol (lib_id "Connector:Screw_Terminal_01x02") (at 43.18 35.56 180) (unit 1)
-    (in_bom yes) (on_board yes)
-    (property "Reference" "J6" (id 0) (at 43.18 30.48 0))
+  (symbol (lib_name "Screw_Terminal_01x02_1") (lib_id "Connector:Screw_Terminal_01x02") (at 43.18 35.56 180) (unit 1)
+    (in_bom yes) (on_board yes)
+    (property "Reference" "J6" (id 0) (at 43.18 40.64 0))
     (property "Value" "Line IN" (id 1) (at 43.18 38.1 0))
     (property "Footprint" "TerminalBlock:TerminalBlock_bornier-2_P5.08mm" (id 2) (at 43.18 35.56 0)
@@
     (pin "1")
   )
+  (symbol (lib_name "Screw_Terminal_01x02_1") (lib_id "Connector:Screw_Terminal_01x02") (at 43.18 48.26 180) (unit 1)
+    (in_bom yes) (on_board yes)
+    (property "Reference" "J7" (id 0) (at 43.18 53.34 0))
+    (property "Value" "Line IN" (id 1) (at 43.18 50.8 0))
+    (property "Footprint" "TerminalBlock:TerminalBlock_bornier-2_P5.08mm" (id 2) (at 43.18 48.26 0)
+      (effects (font (size 1.27 1.27)) hide)
+    )
+    (property "Datasheet" "~" (id 3) (at 43.18 48.26 0)
+      (effects (font (size 1.27 1.27)) hide)
+    )
+    (pin "1")
+    (pin "2")
+  )
   (symbol (lib_id "Device:R") (at 71.12 115.57 90) (unit 1)
     (in_bom yes) (on_board yes)
@@
     (pin "2")
   )
+  (symbol (lib_id "Connector:TestPoint") (at 114.3 92.71 0) (unit 1)
+    (in_bom yes) (on_board yes)
+    (property "Reference" "TP?" (id 0) (at 113.03 87.63 0)
+      (effects (font (size 1.27 1.27)) (justify left))
+    )
+    (property "Value" "Csense_B" (id 1) (at 115.57 90.17 0)
+      (effects (font (size 1.27 1.27)) (justify left))
+    )
+    (property "Footprint" "" (id 2) (at 119.38 92.71 0)
+      (effects (font (size 1.27 1.27)) hide)
+    )
+    (property "Datasheet" "~" (id 3) (at 119.38 92.71 0)
+      (effects (font (size 1.27 1.27)) hide)
+    )
+    (pin "1")
+  )
   (symbol (lib_id "power:VAC") (at 24.13 167.64 0) (unit 1)
     (in_bom yes) (on_board yes)
@@
     (pin "1")
   )
-  (symbol (lib_id "Connector:Screw_Terminal_01x02") (at 43.18 48.26 180) (unit 1)
-    (in_bom yes) (on_board yes)
-    (property "Reference" "J7" (id 0) (at 43.18 43.18 0))
-    (property "Value" "Heater_A" (id 1) (at 43.18 50.8 0))
-    (property "Footprint" "TerminalBlock:TerminalBlock_bornier-2_P5.08mm" (id 2) (at 43.18 48.26 0)
-      (effects (font (size 1.27 1.27)) hide)
-    )
-    (property "Datasheet" "~" (id 3) (at 43.18 48.26 0)
-      (effects (font (size 1.27 1.27)) hide)
-    )
-    (pin "1")
-    (pin "2")
-  )
   (symbol (lib_id "Device:R") (at 194.31 128.27 270) (unit 1)
