File: Electrical/pcb/reflow_oven/reflow_oven.kicad_pcb (KiCad board)
At the start: 2 copper layers, 189 parts, among them J1 1711738, J10 THC IN, J11 THC IN, J12 NTC_A IN, J13 NTC_B IN, J14 3V3 out, J15 5V out, J16 SSR_A, J17 FAN power in, J18 FAN out, J19 SSR_B, J2 Conn_01x06, J3 USER BOARD DISPLAY, J4 USER BOARD BUTTON, J5 DB9_Female_MountingHoles, J6 Line IN, J7 Line IN, J8 Line IN, J9 Heater_B, P1 USB_C_Receptacle_USB2.0, Q1 DMN13H750S, Q2 AO3402, Q3 DMN13H750S, SW1 SW_MEC_5E, T1 ZMPT101B, T2 ZMPT101B, U1 LH05-10B05, U10 TLP2361, U11 COS6001, U12 COS6001, U13 COS6001, U14 COS6001, U2 AP1117-33, U3 STM32F030CCTx, U4 CP2102N-Axx-xQFN28, U5 MAX485E, U6 MAX6675ISA+T, U7 MAX6675ISA+T, U8 ACS758LCB-050B-PFF, U9 ACS758LCB-050B-PFF, Y1 8MHz 8pF

Commit message: production candidate
finished routing
Parts:
- added D18: DSS34, Diode_SMD:D_SOD-123F, F.Cu at (270.6, 102.2)
- added REF**: bolt, footprint_lib:bolt, F.Cu at (267.6, 91.0)
- added REF**: bolt, footprint_lib:bolt, F.Cu at (186.4, 129.7)
- added REF**: Symbol_HighVoltage_Type2_CopperTop_VerySmall, Symbol:Symbol_HighVoltage_Type2_CopperTop_VerySmall, F.Cu at (221.4, 204.7)
- added REF**: bolt, footprint_lib:bolt, F.Cu at (169.1, 213.4)
- added REF**: Symbol_HighVoltage_Type2_CopperTop_VerySmall, Symbol:Symbol_HighVoltage_Type2_CopperTop_VerySmall, F.Cu at (267.8, 204.6)
- added REF**: bolt, footprint_lib:bolt, F.Cu at (174.1, 181.4)
- added REF**: OSHW-Logo_11.4x12mm_SilkScreen, Symbol:OSHW-Logo_11.4x12mm_SilkScreen, F.Cu at (236.5, 125.2)
- added REF**: bolt, footprint_lib:bolt, F.Cu at (280.7, 185.3)
- added REF**: bolt, footprint_lib:bolt, F.Cu at (253.2, 132.5)
- added REF**: bolt, footprint_lib:bolt, F.Cu at (175.2, 91.5)
- added TP1: Csense_A, TestPoint:TestPoint_Pad_D1.5mm, F.Cu at (219.3, 164.6)
- added TP10: B, TestPoint:TestPoint_Pad_D1.5mm, F.Cu at (220.3, 109.1)
- added TP11: A, TestPoint:TestPoint_Pad_D1.5mm, F.Cu at (217.7, 109.1)
- added TP12: ZC_led, TestPoint:TestPoint_Pad_D1.5mm, F.Cu at (181.8, 188.8)
- added TP13: ZC_out, TestPoint:TestPoint_Pad_D1.5mm, F.Cu at (183.1, 167.7)
- added TP14: NTC_A, TestPoint:TestPoint_Pad_D1.5mm, F.Cu at (270.7, 153.7)
- added TP15: VA_op1, TestPoint:TestPoint_Pad_D1.5mm, F.Cu at (189.6, 154.8)
- added TP16: VB_op1, TestPoint:TestPoint_Pad_D1.5mm, F.Cu at (235.9, 154.8)
- added TP17: NTC_B, TestPoint:TestPoint_Pad_D1.5mm, F.Cu at (270.7, 145.8)
- added TP18: Vsense_A, TestPoint:TestPoint_Pad_D1.5mm, F.Cu at (193.4, 154.8)
- added TP19: Vsense_B, TestPoint:TestPoint_Pad_D1.5mm, F.Cu at (239.7, 154.8)
- added TP2: Csense_B, TestPoint:TestPoint_Pad_D1.5mm, F.Cu at (265.7, 164.6)
- added TP3: I2C_SCL, TestPoint:TestPoint_Pad_D1.5mm, F.Cu at (246.8, 113.1)
- added TP4: I2C_SDA, TestPoint:TestPoint_Pad_D1.5mm, F.Cu at (258.4, 110.7)
- added TP5: FAN_GATE, TestPoint:TestPoint_Pad_D1.5mm, F.Cu at (261.0, 99.4)
- added TP6: USBS_RX, TestPoint:TestPoint_Pad_D1.5mm, F.Cu at (199.6, 105.0)
- added TP7: USBS_TX, TestPoint:TestPoint_Pad_D1.5mm, F.Cu at (199.6, 107.7)
- added TP8: 485_RX, TestPoint:TestPoint_Pad_D1.5mm, F.Cu at (232.6, 106.7)
- added TP9: 485_TX, TestPoint:TestPoint_Pad_D1.5mm, F.Cu at (232.6, 103.7)
- added kibuzzard-64E4F476: G***, kibuzzard-64E4F476, F.Cu at (207.8, 204.9)
- added kibuzzard-64E4F49B: G***, kibuzzard-64E4F49B, F.Cu at (254.6, 204.9)
- added kibuzzard-64E4F882: G***, kibuzzard-64E4F882, F.Cu at (282.9, 158.0)
- added kibuzzard-64E4F8B7: G***, kibuzzard-64E4F8B7, F.Cu at (282.9, 149.4)
- added kibuzzard-64E4F997: G***, kibuzzard-64E4F997, F.Cu at (228.0, 221.0)
- added kibuzzard-64E4F997: G***, kibuzzard-64E4F997, F.Cu at (274.2, 221.0)
- added kibuzzard-64E4F9A0: G***, kibuzzard-64E4F9A0, F.Cu at (261.5, 221.0)
- added kibuzzard-64E4F9A0: G***, kibuzzard-64E4F9A0, F.Cu at (215.3, 221.0)
- added kibuzzard-64E4F9DC: G***, kibuzzard-64E4F9DC, F.Cu at (149.5, 221.0)
- added kibuzzard-64E4FDFA: G***, kibuzzard-64E4FDFA, F.Cu at (182.8, 219.0)
- added kibuzzard-64E4FE01: G***, kibuzzard-64E4FE01, F.Cu at (182.8, 215.4)
- added kibuzzard-64E50110: G***, kibuzzard-64E50110, F.Cu at (139.1, 93.8)
- added kibuzzard-64E5011B: G***, kibuzzard-64E5011B, F.Cu at (139.1, 100.9)
- added kibuzzard-64E50301: G***, kibuzzard-64E50301, F.Cu at (157.0, 90.9)
- added kibuzzard-64E50E47: G***, kibuzzard-64E50E47, F.Cu at (191.1, 97.1)
- added kibuzzard-64E5CE1E: G***, kibuzzard-64E5CE1E, F.Cu at (282.6, 129.1)
- added kibuzzard-64E5CE2C: G***, kibuzzard-64E5CE2C, F.Cu at (282.6, 137.7)
- added kibuzzard-64E5FA1C: G***, kibuzzard-64E5FA1C, F.Cu at (264.1, 112.1)
- added kibuzzard-64E5FA1C: G***, kibuzzard-64E5FA1C, F.Cu at (264.1, 120.3)
- added kibuzzard-64E5FC4C: G***, kibuzzard-64E5FC4C, F.Cu at (282.6, 118.9)
- added kibuzzard-64E5FC57: G***, kibuzzard-64E5FC57, F.Cu at (282.6, 110.7)
- added kibuzzard-64E5FCEC: G***, kibuzzard-64E5FCEC, F.Cu at (282.6, 94.4)
- added kibuzzard-64E602C4: G***, kibuzzard-64E602C4, F.Cu at (282.6, 102.2)
- added kibuzzard-64E607E3: G***, kibuzzard-64E607E3, F.Cu at (203.2, 136.7)
- added kibuzzard-64E610EC: G***, kibuzzard-64E610EC, F.Cu at (203.2, 130.3)
- added kibuzzard-64E624F7: G***, kibuzzard-64E624F7, F.Cu at (204.2, 102.8)
- added kibuzzard-64E6252A: G***, kibuzzard-64E6252A, F.Cu at (240.7, 110.6)
- added kibuzzard-64E625F5: G***, kibuzzard-64E625F5, F.Cu at (252.2, 110.6)
- added kibuzzard-64E62979: G***, kibuzzard-64E62979, F.Cu at (203.8, 114.2)
- added kibuzzard-64E62C67: G***, kibuzzard-64E62C67, F.Cu at (253.5, 123.7)
- C26, C27, C32, C33: value 1n -> 1nF
- D9: value D_TVS 5V -> 3V3; footprint Diode_SMD:D_SOD-523 -> Diode_SMD:D_SOD-123
- J7: value Line IN -> Heater_A
- R72: value 10K -> 0
- Y1: footprint Crystal:Crystal_SMD_TXC_7M-4Pin_3.2x2.5mm_HandSoldering -> Crystal:Crystal_SMD_TXC_7M-4Pin_3.2x2.5mm
- moved F7 346.2 mm to (248.5, 215.4), turned to 180 degrees
- moved R34 340.1 mm to (241.9, 213.9), turned to 90 degrees
- moved R37 329.1 mm to (241.9, 207.3), turned to 90 degrees
- moved R40 326.3 mm to (239.1, 202.0), turned to 180 degrees
- moved R44 314.9 mm to (236.9, 196.7), turned to -90 degrees
- moved T2 297.8 mm to (236.9, 185.6), turned to 90 degrees
- moved J9 275.7 mm to (271.8, 215.5)
- moved R48 274.9 mm to (248.1, 165.3), turned to 180 degrees
- moved R33 274.8 mm to (195.6, 213.9), turned to 90 degrees
- moved J8 271.0 mm to (259.1, 215.4)
- moved C24 268.7 mm to (243.3, 165.3), turned to 180 degrees
- moved R36 267.1 mm to (195.6, 207.3), turned to 90 degrees
- moved R55 263.9 mm to (252.0, 164.5), turned to -90 degrees
- moved R51 262.3 mm to (242.4, 162.2), turned to -90 degrees
- moved R57 261.5 mm to (245.9, 162.2), turned to 90 degrees
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Connections:
- net VAC renamed LINE
- C1 pad 2: Net-(C1-Pad2) -> NEUT
- C21 pad 1: VDDA -> +3V3
- C21 pad 2: GNDA -> GND
- C22 pad 1: VDDA -> +3V3
- C22 pad 2: GNDA -> GND
- D8 pad 4: GNDREF -> NEUT
- D9 pad 1: Net-(D8-Pad2) -> Net-(D9-Pad1)
- D9 pad 2: Net-(D9-Pad2) -> Net-(D8-Pad2)
- J1 pad 2: Net-(C1-Pad2) -> NEUT
- J10 pad 1: Net-(J10-Pad1) -> GND
- J10 pad 2: GNDA -> Net-(J10-Pad2)
- J11 pad 1: Net-(J11-Pad1) -> GND
- J11 pad 2: GNDA -> Net-(J11-Pad2)
- J18 pad 1: Net-(J18-Pad1) -> Net-(D18-Pad2)
- J18 pad 2: Net-(J18-Pad2) -> Net-(D18-Pad1)
- J8 pad 1: Net-(J8-Pad1) -> Net-(F7-Pad1)
- J8 pad 2: Net-(F7-Pad1) -> Net-(J8-Pad2)
- J9 pad 1: Net-(J9-Pad1) -> Net-(J8-Pad2)
- J9 pad 2: Net-(J8-Pad1) -> Net-(J9-Pad2)
- JP1 pad 2: VDD -> +3V3
- JP2 pad 1: Net-(J18-Pad2) -> Net-(D18-Pad2)
- JP2 pad 2: Net-(J18-Pad1) -> Net-(D18-Pad1)
- Q2 pad 3: Net-(J18-Pad2) -> Net-(D18-Pad2)
- R3 pad 1: VDD -> +3V3
- R38 pad 2: Net-(D9-Pad2) -> Net-(D9-Pad1)
- R4 pad 1: VDD -> +3V3
- R41 pad 1: VDDA -> +3V3
- R42 pad 1: VDDA -> +3V3
- R72 pad 2: Net-(J18-Pad1) -> Net-(D18-Pad1)
- R9 pad 1: VDD -> +3V3
- RV2 pad 1: Net-(C1-Pad2) -> NEUT
- T2 pad 2: Net-(J8-Pad1) -> Net-(J8-Pad2)
- U1 pad 2: Net-(C1-Pad2) -> NEUT
- U10 pad 1: Net-(D9-Pad2) -> Net-(D9-Pad1)
- U3 pad 11: /Sensors/Vsense_B -> /Sensors/Csense_A
- U3 pad 13: /Interfaces/RX_MCU_usb -> /Interfaces/RX_MCU_485
- U3 pad 14: /Sensors/Csense_A -> /Sensors/Vsense_B
- U3 pad 31: /Interfaces/RX_MCU_485 -> /Interfaces/RX_MCU_usb
- U3 pad 38: /Actuation/SSR_B -> /Actuation/SSR_A
- U3 pad 39: /Actuation/SSR_A -> /Actuation/SSR_B
- U6 pad 1: GNDA -> GND
- U6 pad 2: GNDA -> GND
- U6 pad 3: Net-(J10-Pad1) -> Net-(J10-Pad2)
- U6 pad 4: VDDA -> +3V3
- U7 pad 1: GNDA -> GND
- U7 pad 2: GNDA -> GND
- U7 pad 3: Net-(J11-Pad1) -> Net-(J11-Pad2)
- U7 pad 4: VDDA -> +3V3
- U9 pad 5: Net-(J9-Pad1) -> Net-(J9-Pad2)
- Y1 pad 3: /MCU_User/OSC_OUT -> Net-(C7-Pad1)
Routing:
- net +5V: track 0.00 -> 166.4 mm, vias 0 -> 1
- net NEUT: track 0.00 -> 100.4 mm
- net /Actuation/FAN: track 0.00 -> 71.4 mm, vias 0 -> 4
- net /MCU_User/I2C1_SDA: track 0.00 -> 68.9 mm, vias 0 -> 4
- net +3V3: track 0.00 -> 68.0 mm, vias 0 -> 44
- net /Sensors/Csense_B: track 0.00 -> 67.6 mm, vias 0 -> 2
- net /Interfaces/RX_MCU_usb: track 0.00 -> 66.9 mm, vias 0 -> 4
- net /MCU_User/I2C1_SCL: track 0.00 -> 66.3 mm, vias 0 -> 4
- net /Interfaces/TX_MCU_usb: track 0.00 -> 65.4 mm, vias 0 -> 4
- net /MCU_User/SPI_CLK: track 0.00 -> 64.8 mm, vias 0 -> 3
- net /MCU_User/SPI_MISO: track 0.00 -> 64.6 mm, vias 0 -> 3
- net GNDREF: track 0.00 -> 63.9 mm
- net /MCU_User/NTC_A: track 0.00 -> 60.6 mm
- net /Actuation/SSR_B: track 0.00 -> 59.9 mm, vias 0 -> 2
- net VBUS: track 0.00 -> 59.2 mm, vias 0 -> 2
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- added copper zone on B.Cu, net +3V3
- added copper zone on F.Cu, net GND
- added copper zone on B.Cu, net GNDA
- added copper zone on B.Cu, net Net-(F6-Pad1)
- added copper zone on F.Cu, net Net-(F6-Pad1)
- added copper zone on B.Cu, net Net-(F7-Pad1)
- added copper zone on F.Cu, net Net-(F7-Pad1)
- added copper zone on B.Cu, net Net-(J6-Pad2)
- added copper zone on F.Cu, net Net-(J6-Pad2)
- added copper zone on B.Cu, net Net-(J7-Pad2)
- added copper zone on F.Cu, net Net-(J7-Pad2)
- added copper zone on B.Cu, net Net-(J8-Pad2)
- added copper zone on F.Cu, net Net-(J8-Pad2)
- added copper zone on B.Cu, net Net-(J9-Pad2)
- added copper zone on F.Cu, net Net-(J9-Pad2)
- added copper zone on B.Cu, net VDD
- added copper zone on F.Cu, net VDDA
Other:
- board outline added: 146.1 x 134.4 mm
- board text added: "+"
- board text added: "-"
- board text added: "3V3"
- board text added: "A"
- board text added: "B"
- board text added: "D"
- board text added: "GND"
- board text added: "H+"
- board text added: "H-"
- board text added: "JLCJLCJLCJLC"
- board text added: "NRST"
- board text added: "SWCLK"
- board text added: "SWDIO"

Commit message: fab out
added fabrication output
Other:
- board text added: "BUZZ"
- board text added: "CLK"
- board text added: "CS"
- board text added: "DWN"
- board text added: "LT"
- board text added: "OK"
- board text added: "RST"
- board text added: "RT"
- board text added: "RW"
- board text added: "SCL"
- board text added: "SDA"
- board text added: "UP"
