File: Electrical/pcb/reflow_oven/Actuation.kicad_sch (KiCad schematic)
At the start: 23 parts, among them J16 SSR_A, J17 FAN power in, J18 FAN out, J19 SSR_B, Q1 DMN13H750S, Q2 AO3402, Q3 DMN13H750S

Commit message: addon
documentation pics
adjust oshw logo
Parts:
- D18: value DSS34 -> BAS85
- TP5: now left out of the parts list
Changed lines of the file:
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@@
       (effects (font (size 1.27 1.27)) hide)
     )
-    (pin "2")
-    (pin "1")
+    (pin "1")
+    (pin "2")
   )
   (symbol (lib_id "power:GND") (at 64.77 76.2 0) (unit 1)
@@
     (in_bom yes) (on_board yes)
     (property "Reference" "D18" (id 0) (at 57.15 116.84 0))
-    (property "Value" "DSS34" (id 1) (at 62.23 116.84 0))
+    (property "Value" "BAS85" (id 1) (at 62.23 116.84 0))
     (property "Footprint" "Diode_SMD:D_SOD-123F" (id 2) (at 59.69 116.84 0)
       (effects (font (size 1.27 1.27)) hide)
@@
   )
   (symbol (lib_id "Connector:TestPoint") (at 55.88 125.73 0) (unit 1)
-    (in_bom yes) (on_board yes)
+    (in_bom no) (on_board yes)
     (property "Reference" "TP5" (id 0) (at 54.61 120.65 0)
       (effects (font (size 1.27 1.27)) (justify left))
@@
       (effects (font (size 1.27 1.27)) hide)
     )
-    (pin "2")
-    (pin "1")
+    (pin "1")
+    (pin "2")
   )
   (symbol (lib_id "Device:R") (at 64.77 40.64 180) (unit 1)

Commit message: documentazione
aggiunta documentazione
Changed lines of the file:
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@@
     (effects (font (size 1.27 1.27)) (justify left bottom))
   )
-  (text "SSR Enable" (at 26.67 30.48 0)
+  (text "SSR Enable" (at 15.875 20.32 0)
     (effects (font (size 2 2) (thickness 0.4) bold) (justify left bottom))
   )
