File: Electrical/pcb/reflow_oven/MCU_User.kicad_sch (KiCad schematic)
At the start: 25 parts, among them J2 Conn_01x06, SW1 SW_MEC_5E, U3 STM32F030CCTx, Y1 8MHz 8pF

Commit message: addon
documentation pics
adjust oshw logo
Parts:
- TP3, TP4: now left out of the parts list
Changed lines of the file:
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@@
   )
   (symbol (lib_id "Connector:TestPoint") (at 45.72 86.36 0) (unit 1)
-    (in_bom yes) (on_board yes)
+    (in_bom no) (on_board yes)
     (property "Reference" "TP4" (id 0) (at 44.45 81.28 0)
       (effects (font (size 1.27 1.27)) (justify left))
@@
   )
   (symbol (lib_id "Connector:TestPoint") (at 34.29 86.36 0) (unit 1)
-    (in_bom yes) (on_board yes)
+    (in_bom no) (on_board yes)
     (property "Reference" "TP3" (id 0) (at 33.02 81.28 0)
       (effects (font (size 1.27 1.27)) (justify left))

Commit message: addon
test nucleo f746
Other:
- note added: "DNP"
Changed lines of the file:
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@@
     (effects (font (size 1.27 1.27)) (justify left bottom))
+  )
+  (text "DNP" (at 34.29 61.595 270)
+    (effects (font (size 1.27 1.27)) (justify right bottom))
   )
   (text "Oscillator" (at 25.4 116.84 0)
     (effects (font (size 2 2) (thickness 0.4) bold) (justify left bottom))
   )
+  (text "DNP" (at 46.99 61.595 270)
+    (effects (font (size 1.27 1.27)) (justify right bottom))
+  )
   (label "OSC_IN" (at 195.58 57.15 0)

Commit message: documentazione
aggiunta documentazione
Changed lines of the file:
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@@
     (effects (font (size 1.27 1.27)) (justify left bottom))
   )
-  (text "Non-standard connetion" (at 104.14 73.66 0)
+  (text "Non-standard connetion" (at 104.14 80.01 0)
     (effects (font (size 1.27 1.27)) (justify left bottom))
   )
